Commit message: merge UR10+Robotiq, author SRDF, fix viser mesh-scale bug
Combined arm: merge_ur10_robotiq.py stitches the two separately-vendored
URDFs at tool0 (mount offset placeholder, not yet visually verified) with
a gripper_tcp reference frame 0.15m along the gripper's local +Z (also a
placeholder). ur10_robotiq.srdf authored fresh (neither upstream ships
HPP semantics) — <gripper> at gripper_tcp per the panda_bimanual.srdf
precedent, plus a first-pass disable_collisions list for the finger
linkage.

Hit a real bug getting this into viser: Robotiq's meshes are authored in
millimeters (<mesh scale="0.001 0.001 0.001"/>), which triggers the
already-documented pyhpp_viser bug (see pokeball_bimanual.urdf's own
comment) where rendered position = world_translation * meshScale instead
of only scaling local vertices — collapsed the whole gripper to within
~1mm of world origin regardless of its real pose, while UR10 (unit scale,
unaffected) rendered correctly but off-frame. Fixed the same way the
pokeball example already did: rescale_robotiq_meshes.py bakes the 0.001
factor into the mesh vertices via trimesh (meshes_scaled/), eliminating
the non-unit <mesh scale> entirely — confirmed via FK dump that every
geometry now has meshScale=[1,1,1].

view_arm_gripper.py loads the combined arm alone in viser for visual
verification (arm+gripper only, no table/second arm yet). Also surfaced
an unrelated pre-existing bug: PyHPPBackend.neutral_config() calls
Device.neutralConfiguration(), which doesn't exist on this pyhpp
version — routed around it with device.currentConfiguration() directly,
noted inline, not fixed at the source (out of scope for this branch).

File: script/ikea_table_prototype/assets/robotiq_2f85/urdf/robotiq_2f85_generated.urdf (robot description, URDF)
Before this commit: robot robotiq_arg2f_85_model, 11 links, 10 joints
Links:
- link left_inner_finger: geometry collision mesh filename=/Users/thanhndv212/Develop/agimus-ws/long-tamp/script/ikea_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; visual mesh filename=/Users/thanhndv212/Develop/agimus-ws/long-tamp/script/ikea_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
- link left_inner_knuckle: geometry collision mesh filename=/Users/thanhndv212/Develop/agimus-ws/long-tamp/script/ikea_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; visual mesh filename=/Users/thanhndv212/Develop/agimus-ws/long-tamp/script/ikea_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
- link left_outer_finger: geometry collision mesh filename=/Users/thanhndv212/Develop/agimus-ws/long-tamp/script/ikea_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; visual mesh filename=/Users/thanhndv212/Develop/agimus-ws/long-tamp/script/ikea_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
- link left_outer_knuckle: geometry collision mesh filename=/Users/thanhndv212/Develop/agimus-ws/long-tamp/script/ikea_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; visual mesh filename=/Users/thanhndv212/Develop/agimus-ws/long-tamp/script/ikea_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
- link right_inner_finger: geometry collision mesh filename=/Users/thanhndv212/Develop/agimus-ws/long-tamp/script/ikea_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; visual mesh filename=/Users/thanhndv212/Develop/agimus-ws/long-tamp/script/ikea_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
- link right_inner_knuckle: geometry collision mesh filename=/Users/thanhndv212/Develop/agimus-ws/long-tamp/script/ikea_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; visual mesh filename=/Users/thanhndv212/Develop/agimus-ws/long-tamp/script/ikea_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
- link right_outer_finger: geometry collision mesh filename=/Users/thanhndv212/Develop/agimus-ws/long-tamp/script/ikea_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; visual mesh filename=/Users/thanhndv212/Develop/agimus-ws/long-tamp/script/ikea_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
- link right_outer_knuckle: geometry collision mesh filename=/Users/thanhndv212/Develop/agimus-ws/long-tamp/script/ikea_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; visual mesh filename=/Users/thanhndv212/Develop/agimus-ws/long-tamp/script/ikea_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
- link robotiq_arg2f_base_link: geometry collision mesh filename=/Users/thanhndv212/Develop/agimus-ws/long-tamp/script/ikea_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; visual mesh filename=/Users/thanhndv212/Develop/agimus-ws/long-tamp/script/ikea_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

File: script/ikea_table_prototype/assets/robotiq_2f85/urdf/robotiq_arg2f.xacro (robot description, xacro)
@@ -11,5 +11,5 @@
         <origin xyz="0 0 0" rpy="0 0 0" />
         <geometry>
-          <mesh filename="/Users/thanhndv212/Develop/agimus-ws/long-tamp/script/ikea_table_prototype/assets/robotiq_2f85/meshes/visual/robotiq_arg2f_85_base_link.dae" scale="0.001 0.001 0.001"/>
+          <mesh filename="/Users/thanhndv212/Develop/agimus-ws/long-tamp/script/ikea_table_prototype/assets/robotiq_2f85/meshes_scaled/visual/robotiq_arg2f_85_base_link.dae"/>
         </geometry>
         <material name="">
@@ -20,5 +20,5 @@
         <origin xyz="0 0 0" rpy="0 0 0" />
         <geometry>
-           <mesh filename="/Users/thanhndv212/Develop/agimus-ws/long-tamp/script/ikea_table_prototype/assets/robotiq_2f85/meshes/collision/robotiq_arg2f_base_link.stl" />
+           <mesh filename="/Users/thanhndv212/Develop/agimus-ws/long-tamp/script/ikea_table_prototype/assets/robotiq_2f85/meshes_scaled/collision/robotiq_arg2f_base_link.stl" />
         </geometry>
       </collision>

File: script/ikea_table_prototype/assets/robotiq_2f85/urdf/robotiq_arg2f_85_model_macro.xacro (robot description, xacro)
@@ -12,5 +12,5 @@
         <origin xyz="0 0 0" rpy="0 0 0" />
         <geometry>
-          <mesh filename="/Users/thanhndv212/Develop/agimus-ws/long-tamp/script/ikea_table_prototype/assets/robotiq_2f85/meshes/visual/robotiq_arg2f_85_outer_knuckle.dae" scale="0.001 0.001 0.001"/>
+          <mesh filename="/Users/thanhndv212/Develop/agimus-ws/long-tamp/script/ikea_table_prototype/assets/robotiq_2f85/meshes_scaled/visual/robotiq_arg2f_85_outer_knuckle.dae"/>
         </geometry>
         <material name="">
@@ -21,5 +21,5 @@
         <origin xyz="0 0 0" rpy="0 0 0" />
         <geometry>
-          <mesh filename="/Users/thanhndv212/Develop/agimus-ws/long-tamp/script/ikea_table_prototype/assets/robotiq_2f85/meshes/collision/robotiq_arg2f_85_outer_knuckle.dae" scale="0.001 0.001 0.001"/>
+          <mesh filename="/Users/thanhndv212/Develop/agimus-ws/long-tamp/script/ikea_table_prototype/assets/robotiq_2f85/meshes_scaled/collision/robotiq_arg2f_85_outer_knuckle.dae"/>
         </geometry>
       </collision>
@@ -36,5 +36,5 @@
         <origin xyz="0 0 0" rpy="0 0 0" />
         <geometry>
-          <mesh filename="/Users/thanhndv212/Develop/agimus-ws/long-tamp/script/ikea_table_prototype/assets/robotiq_2f85/meshes/visual/robotiq_arg2f_85_outer_finger.dae" scale="0.001 0.001 0.001"/>
+          <mesh filename="/Users/thanhndv212/Develop/agimus-ws/long-tamp/script/ikea_table_prototype/assets/robotiq_2f85/meshes_scaled/visual/robotiq_arg2f_85_outer_finger.dae"/>
         </geometry>
         <material name="">
@@ -45,5 +45,5 @@
         <origin xyz="0 0 0" rpy="0 0 0" />
         <geometry>
-          <mesh filename="/Users/thanhndv212/Develop/agimus-ws/long-tamp/script/ikea_table_prototype/assets/robotiq_2f85/meshes/collision/robotiq_arg2f_85_outer_finger.dae" scale="0.001 0.001 0.001"/>
+          <mesh filename="/Users/thanhndv212/Develop/agimus-ws/long-tamp/script/ikea_table_prototype/assets/robotiq_2f85/meshes_scaled/collision/robotiq_arg2f_85_outer_finger.dae"/>
         </geometry>
       </collision>
@@ -60,5 +60,5 @@
         <origin xyz="0 0 0" rpy="0 0 0" />
         <geometry>
-          <mesh filename="/Users/thanhndv212/Develop/agimus-ws/long-tamp/script/ikea_table_prototype/assets/robotiq_2f85/meshes/visual/robotiq_arg2f_85_inner_knuckle.dae" scale="0.001 0.001 0.001"/>
+          <mesh filename="/Users/thanhndv212/Develop/agimus-ws/long-tamp/script/ikea_table_prototype/assets/robotiq_2f85/meshes_scaled/visual/robotiq_arg2f_85_inner_knuckle.dae"/>
         </geometry>
         <material name="">
@@ -69,5 +69,5 @@
         <origin xyz="0 0 0" rpy="0 0 0" />
         <geometry>
-          <mesh filename="/Users/thanhndv212/Develop/agimus-ws/long-tamp/script/ikea_table_prototype/assets/robotiq_2f85/meshes/collision/robotiq_arg2f_85_inner_knuckle.dae" scale="0.001 0.001 0.001"/>
+          <mesh filename="/Users/thanhndv212/Develop/agimus-ws/long-tamp/script/ikea_table_prototype/assets/robotiq_2f85/meshes_scaled/collision/robotiq_arg2f_85_inner_knuckle.dae"/>
         </geometry>
       </collision>
@@ -84,5 +84,5 @@
         <origin xyz="0 0 0" rpy="0 0 0" />
         <geometry>
-          <mesh filename="/Users/thanhndv212/Develop/agimus-ws/long-tamp/script/ikea_table_prototype/assets/robotiq_2f85/meshes/visual/robotiq_arg2f_85_inner_finger.dae" scale="0.001 0.001 0.001"/>
+          <mesh filename="/Users/thanhndv212/Develop/agimus-ws/long-tamp/script/ikea_table_prototype/assets/robotiq_2f85/meshes_scaled/visual/robotiq_arg2f_85_inner_finger.dae"/>
         </geometry>
         <material name="">
@@ -93,5 +93,5 @@
         <origin xyz="0 0 0" rpy="0 0 0" />
         <geometry>
-          <mesh filename="/Users/thanhndv212/Develop/agimus-ws/long-tamp/script/ikea_table_prototype/assets/robotiq_2f85/meshes/collision/robotiq_arg2f_85_inner_finger.dae" scale="0.001 0.001 0.001" />
+          <mesh filename="/Users/thanhndv212/Develop/agimus-ws/long-tamp/script/ikea_table_prototype/assets/robotiq_2f85/meshes_scaled/collision/robotiq_arg2f_85_inner_finger.dae" />
         </geometry>
       </collision>
