Commit message: give the workbench actual support legs
First pass was just the tabletop slab (z=0.36 to 0.40) with nothing
under it down to the ground — same "floating in mid-air" problem the
workbench itself was supposed to fix, one level up. Added 4 identical
box legs at the footprint's corners (inset 0.05m), spanning z=0
(ground) to z=0.36 (slab underside). Validated the URDF parses (5
visual geoms: slab + 4 legs) before relaunching; FK placement check
still confirms table/legs land exactly on the (unchanged) surface
height.

File: script/ikea_table_prototype/generated/workbench.urdf (robot description, URDF)
Before this commit: robot workbench, 1 links, 0 joints
Links:
- link workbench_base: geometry collision box size=0.05 0.05 0.36; collision box size=0.05 0.05 0.36
