Commit message: rescale table/leg meshes too — same pyhpp_viser bug, third hit
"no not yet" after the recentering commit — table/legs still weren't
where they should be, even though the underlying model data (FK,
q values) was already confirmed correct. Root-caused with the same
live-introspection technique used for the pedestal bug:
backend.viewer._visual_geometry_frames showed table/leg cached
positions that were each exactly target_position * mesh_scale (e.g.
table target (0.75, 0, 0.5) cached as (0.01125, 0, 0.01) =
(0.75*0.015, 0, 0.5*0.02)) — the same "rendered position =
world_translation * meshScale" bug as the Robotiq gripper fix
earlier in this branch, this time triggered by generate_urdf_srdf.py
giving the raw IKEA STLs a non-unit <mesh scale> (0.015/0.015/0.02
for the table, 0.02/0.02/0.02 for the legs) to bring them to meters.

Fix, same pattern as rescale_robotiq_meshes.py: rescale_ikea_meshes.py
bakes those factors into the mesh vertices via trimesh
(meshes_scaled/), generate_urdf_srdf.py now points there with
mesh_scale="1 1 1" (a no-op) instead. Verified via the same live
introspection: all 5 cached positions now match their targets
exactly.

File: script/ikea_table_prototype/generated/leg1.urdf (robot description, URDF)
Before this commit: robot leg1, 1 links, 0 joints
Links:
- link base_link: geometry collision box size=0.03 0.03 0.2625; visual mesh filename=/home/thanhndv212/devel/hpp/src/long_tamp/script/ikea_table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 scale=1 1 1

File: script/ikea_table_prototype/generated/leg2.urdf (robot description, URDF)
Before this commit: robot leg2, 1 links, 0 joints
Links:
- link base_link: geometry collision box size=0.03 0.03 0.2625; visual mesh filename=/home/thanhndv212/devel/hpp/src/long_tamp/script/ikea_table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 scale=1 1 1

File: script/ikea_table_prototype/generated/leg3.urdf (robot description, URDF)
Before this commit: robot leg3, 1 links, 0 joints
Links:
- link base_link: geometry collision box size=0.03 0.03 0.2625; visual mesh filename=/home/thanhndv212/devel/hpp/src/long_tamp/script/ikea_table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 scale=1 1 1

File: script/ikea_table_prototype/generated/leg4.urdf (robot description, URDF)
Before this commit: robot leg4, 1 links, 0 joints
Links:
- link base_link: geometry collision box size=0.03 0.03 0.2625; visual mesh filename=/home/thanhndv212/devel/hpp/src/long_tamp/script/ikea_table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 scale=1 1 1

File: script/ikea_table_prototype/generated/table.urdf (robot description, URDF)
Before this commit: robot table, 1 links, 0 joints
Links:
- link base_link: geometry collision box size=0.64 0.24 0.04; visual mesh filename=/home/thanhndv212/devel/hpp/src/long_tamp/script/ikea_table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 scale=1 1 1

Commit message: drop real IKEA meshes from table/leg visuals, plain box instead
The real STL meshes (visual layer) bake in the actual IKEA LACK
table's screw-hole/dowel-hole surface detail, rendering visibly —
not wanted even for local prototyping. Visual geometry is now the
same plain box already used for collision, for both table and legs.

generate_urdf_srdf.py: dropped the now-unused MESH_DIR/TEXTURE
constants and the <mesh filename> branch of URDF_TEMPLATE entirely;
also corrects the module docstring's "regenerate per environment"
caveat, which no longer applies to these two objects (no absolute
mesh paths left in their output at all) — still applies to the
UR10/Robotiq arm URDFs elsewhere in this directory. The vendored STL
files themselves are untouched, just unreferenced.

File: script/ikea_table_prototype/generated/leg1.urdf (robot description, URDF)
Before this commit: robot leg1, 1 links, 0 joints
Links:
- link base_link: geometry collision box size=0.03 0.03 0.2625; visual box size=0.03 0.03 0.2625

File: script/ikea_table_prototype/generated/leg2.urdf (robot description, URDF)
Before this commit: robot leg2, 1 links, 0 joints
Links:
- link base_link: geometry collision box size=0.03 0.03 0.2625; visual box size=0.03 0.03 0.2625

File: script/ikea_table_prototype/generated/leg3.urdf (robot description, URDF)
Before this commit: robot leg3, 1 links, 0 joints
Links:
- link base_link: geometry collision box size=0.03 0.03 0.2625; visual box size=0.03 0.03 0.2625

File: script/ikea_table_prototype/generated/leg4.urdf (robot description, URDF)
Before this commit: robot leg4, 1 links, 0 joints
Links:
- link base_link: geometry collision box size=0.03 0.03 0.2625; visual box size=0.03 0.03 0.2625

File: script/ikea_table_prototype/generated/table.urdf (robot description, URDF)
Before this commit: robot table, 1 links, 0 joints
Links:
- link base_link: geometry collision box size=0.64 0.24 0.04; visual box size=0.64 0.24 0.04

Commit message: real recessed holes + pegs, generated fresh via boolean ops
User wanted actual holes/pegs, not just a flush visual marker. URDF
has no native CSG subtraction for primitives, so
generate_hole_peg_meshes.py builds fresh meshes via trimesh boolean
ops (needed a backend — pip install manifold3d, not present by
default in this HPP env):
- table_with_holes.stl: the table box minus 4 blind cylindrical
  holes at the real socket XY positions (from the reference MJCF),
  0.012m radius, 0.015m deep.
- leg_with_peg.stl: the leg box plus one protruding cylindrical peg
  on the top face, 0.01m radius, 0.02m tall (shared by all 4 legs —
  geometrically identical).

Not derived from the real vendored IKEA STL in any way — built purely
from the box dimensions/socket positions already used for collision.
Verified geometrically before wiring in (point-containment checks:
hole positions are empty space, peg tip is solid, both watertight).

Visual only — collision stays the plain convex box, since HPP-FCL's
narrow-phase checking wants convex shapes and a box-with-holes isn't
(standard practice: detailed visual mesh, simple convex collision
proxy, same as e.g. UR10's own separate visual/collision meshes).
No <mesh scale> needed since these are authored directly in meters.

generate_urdf_srdf.py updated to reference the new meshes; validated
via Pinocchio (loads, 1 visual + 1 collision geom per object) and the
live FK placement check before confirming in viser.

File: script/ikea_table_prototype/generated/leg1.urdf (robot description, URDF)
Before this commit: robot leg1, 1 links, 0 joints
Links:
- link base_link: geometry collision box size=0.03 0.03 0.2625; visual mesh filename=/home/thanhndv212/devel/hpp/src/long_tamp/script/ikea_table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

File: script/ikea_table_prototype/generated/leg2.urdf (robot description, URDF)
Before this commit: robot leg2, 1 links, 0 joints
Links:
- link base_link: geometry collision box size=0.03 0.03 0.2625; visual mesh filename=/home/thanhndv212/devel/hpp/src/long_tamp/script/ikea_table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

File: script/ikea_table_prototype/generated/leg3.urdf (robot description, URDF)
Before this commit: robot leg3, 1 links, 0 joints
Links:
- link base_link: geometry collision box size=0.03 0.03 0.2625; visual mesh filename=/home/thanhndv212/devel/hpp/src/long_tamp/script/ikea_table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

File: script/ikea_table_prototype/generated/leg4.urdf (robot description, URDF)
Before this commit: robot leg4, 1 links, 0 joints
Links:
- link base_link: geometry collision box size=0.03 0.03 0.2625; visual mesh filename=/home/thanhndv212/devel/hpp/src/long_tamp/script/ikea_table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

File: script/ikea_table_prototype/generated/table.urdf (robot description, URDF)
Before this commit: robot table, 1 links, 0 joints
Links:
- link base_link: geometry collision box size=0.64 0.24 0.04; visual mesh filename=/home/thanhndv212/devel/hpp/src/long_tamp/script/ikea_table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

Commit message: feat: Add gripper sliders to the GUI and update leg docking mechanism
- Implemented gripper mimic joint handling in the GUI, allowing for open/close sliders for each arm's gripper.
- Updated leg docking mechanism in SRDF files to use gripper handles instead of placement contacts, ensuring deterministic docking behavior.
- Adjusted URDF files to reflect changes in leg and table geometry, including mesh file paths.
- Enhanced task assembly logic to accommodate new docking approach, ensuring all objects remain present in the task configuration.
- Fixed pedestal dimensions in URDF files for better alignment with the robotic arm setup.

File: script/ikea_table_prototype/generated/leg1.urdf (robot description, URDF)
Before this commit: robot leg1, 1 links, 0 joints
Links:
- link base_link: geometry collision box size=0.03 0.03 0.2625; visual mesh filename=/Users/thanhndv212/Develop/agimus-ws/long-tamp/script/ikea_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

File: script/ikea_table_prototype/generated/leg2.urdf (robot description, URDF)
Before this commit: robot leg2, 1 links, 0 joints
Links:
- link base_link: geometry collision box size=0.03 0.03 0.2625; visual mesh filename=/Users/thanhndv212/Develop/agimus-ws/long-tamp/script/ikea_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

File: script/ikea_table_prototype/generated/leg3.urdf (robot description, URDF)
Before this commit: robot leg3, 1 links, 0 joints
Links:
- link base_link: geometry collision box size=0.03 0.03 0.2625; visual mesh filename=/Users/thanhndv212/Develop/agimus-ws/long-tamp/script/ikea_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

File: script/ikea_table_prototype/generated/leg4.urdf (robot description, URDF)
Before this commit: robot leg4, 1 links, 0 joints
Links:
- link base_link: geometry collision box size=0.03 0.03 0.2625; visual mesh filename=/Users/thanhndv212/Develop/agimus-ws/long-tamp/script/ikea_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

File: script/ikea_table_prototype/generated/table.urdf (robot description, URDF)
Before this commit: robot table, 1 links, 0 joints
Links:
- link base_link: geometry collision box size=0.64 0.24 0.04; visual mesh filename=/Users/thanhndv212/Develop/agimus-ws/long-tamp/script/ikea_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

File: script/ikea_table_prototype/generated/ur10_robotiq.container.urdf (robot description, URDF)
Before this commit: robot ur10_robotiq, 24 links, 23 joints
Links:
- link pedestal: geometry collision box size=0.3 0.3 0.6; visual box size=0.3 0.3 0.6
Joints:
- joint pedestal_to_arm: origin xyz=0 0 0.5 rpy=0 0 0 -> xyz=0 0 0.6 rpy=0 0 0

File: script/ikea_table_prototype/generated/ur10_robotiq.urdf (robot description, URDF)
Before this commit: robot ur10_robotiq, 24 links, 23 joints
Links:
- link pedestal: geometry collision box size=0.3 0.3 0.6; visual box size=0.3 0.3 0.6
Joints:
- joint pedestal_to_arm: origin xyz=0 0 0.5 rpy=0 0 0 -> xyz=0 0 0.6 rpy=0 0 0

File: script/ikea_table_prototype/generated/ur10_robotiq_right.container.urdf (robot description, URDF)
Before this commit: robot ur10_robotiq, 25 links, 24 joints
Links:
- link pedestal: geometry collision box size=0.3 0.3 0.6; visual box size=0.3 0.3 0.6
Joints:
- joint pedestal_to_arm: origin xyz=0 0 0.5 rpy=0 0 0 -> xyz=0 0 0.6 rpy=0 0 0

File: script/ikea_table_prototype/generated/ur10_robotiq_right.urdf (robot description, URDF)
Before this commit: robot ur10_robotiq, 25 links, 24 joints
Links:
- link pedestal: geometry collision box size=0.3 0.3 0.6; visual box size=0.3 0.3 0.6
Joints:
- joint pedestal_to_arm: origin xyz=0 0 0.5 rpy=0 0 0 -> xyz=0 0 0.6 rpy=0 0 0
