Commit message: fold the pedestal into the arm URDF, lower to 0.3m
Per feedback: 0.5m read as too tall, and the separately-positioned
pedestal object could visually gap from the arm even though they were
numerically aligned. merge_ur10_robotiq.py now bakes the pedestal
directly into ur10_robotiq.urdf as a fixed joint onto UR10's own root
("world") — one rigid body, no possibility of misalignment — and
drops the height to 0.3m. view_full_scene.py's arm pose goes back to
z=0 (ground level); the URDF's own pedestal_to_arm joint supplies the
elevation. Removed the now-unused standalone pedestal.urdf.

Verified via Pinocchio frame FK before touching the viewer: pedestal
base at z=0, world/base_link at exactly z=0.3, tool0 correspondingly
higher — confirmed live in viser afterward. Object placement re-
checked too (table + all 4 legs, still exactly on target).

File: script/ikea_table_prototype/generated/ur10_robotiq.container.urdf (robot description, URDF)
Before this commit: robot ur10_robotiq, 23 links, 22 joints
Links:
- added link pedestal; collision box size=0.3 0.3 0.3; visual box size=0.3 0.3 0.3
Joints:
- added joint pedestal_to_arm: type fixed, parent pedestal, child world, origin xyz=0 0 0.3 rpy=0 0 0

File: script/ikea_table_prototype/generated/ur10_robotiq.urdf (robot description, URDF)
Before this commit: robot ur10_robotiq, 23 links, 22 joints
Links:
- added link pedestal; collision box size=0.3 0.3 0.3; visual box size=0.3 0.3 0.3
Joints:
- added joint pedestal_to_arm: type fixed, parent pedestal, child world, origin xyz=0 0 0.3 rpy=0 0 0

Commit message: regenerate leg/table/arm URDF+SRDF via build_assets.py
Output of the new pipeline against config/ikea_table_config.yaml.
ur10_robotiq.srdf also gains the plain-UR10-arm adjacent-pair exclusions
(base_link through wrist_3_link) — the first real planning run hit
"Collision between object ur10_left/shoulder_link_0 and
ur10_left/upper_arm_link_0", a guaranteed false positive between two
links joined directly by shoulder_lift_joint, same as any other adjacent
pair; the file's own prior comment already flagged that only the gripper
linkage had been covered, not the arm chain.

File: script/ikea_table_prototype/generated/ur10_robotiq.container.urdf (robot description, URDF)
Before this commit: robot ur10_robotiq, 24 links, 23 joints
Links:
- link pedestal: geometry collision box size=0.3 0.3 0.5; visual box size=0.3 0.3 0.5
Joints:
- joint pedestal_to_arm: origin xyz=0 0 0.3 rpy=0 0 0 -> xyz=0 0 0.5 rpy=0 0 0

File: script/ikea_table_prototype/generated/ur10_robotiq.urdf (robot description, URDF)
Before this commit: robot ur10_robotiq, 24 links, 23 joints
Links:
- link pedestal: geometry collision box size=0.3 0.3 0.5; visual box size=0.3 0.3 0.5
Joints:
- joint pedestal_to_arm: origin xyz=0 0 0.3 rpy=0 0 0 -> xyz=0 0 0.5 rpy=0 0 0

File: script/ikea_table_prototype/generated/ur10_robotiq_right.container.urdf (robot description, URDF)
Before this commit: robot ur10_robotiq, 25 links, 24 joints
Links:
- link pedestal: geometry collision box size=0.3 0.3 0.5; visual box size=0.3 0.3 0.5
Joints:
- joint pedestal_to_arm: origin xyz=0 0 0.3 rpy=0 0 0 -> xyz=0 0 0.5 rpy=0 0 0

File: script/ikea_table_prototype/generated/ur10_robotiq_right.urdf (robot description, URDF)
Before this commit: robot ur10_robotiq, 25 links, 24 joints
Links:
- link pedestal: geometry collision box size=0.3 0.3 0.5; visual box size=0.3 0.3 0.5
Joints:
- joint pedestal_to_arm: origin xyz=0 0 0.3 rpy=0 0 0 -> xyz=0 0 0.5 rpy=0 0 0

Commit message: feat(examples): the UR10 from Universal Robots' own description package

File: script/ikea_table_prototype/generated/ur10_robotiq.container.urdf (robot description, URDF)
Before this commit: robot ur10_robotiq, 24 links, 23 joints
Links:
- removed link ee_link
- added link base_link_inertia, mass 4.0; collision mesh filename=../assets/ur10/official/meshes/ur10/collision/base.stl; visual mesh filename=../assets/ur10/official/meshes/ur10/visual/base.dae
- added link flange
- added link ft_frame
- link base: mass 0.0 -> None
- link base_link: mass 4.0 -> None; geometry 
- link forearm_link: mass 3.87 -> 4.27; geometry collision mesh filename=../assets/ur10/official/meshes/ur10/collision/forearm.stl; visual mesh filename=../assets/ur10/official/meshes/ur10/visual/forearm.dae
- link shoulder_link: mass 7.778 -> 7.1; geometry collision mesh filename=../assets/ur10/official/meshes/ur10/collision/shoulder.stl; visual mesh filename=../assets/ur10/official/meshes/ur10/visual/shoulder.dae
- link tool0: mass 0.0 -> None
- link upper_arm_link: mass 12.93 -> 12.7; geometry collision mesh filename=../assets/ur10/official/meshes/ur10/collision/upperarm.stl; visual mesh filename=../assets/ur10/official/meshes/ur10/visual/upperarm.dae
- link wrist_1_link: mass 1.96 -> 2.0; geometry collision mesh filename=../assets/ur10/official/meshes/ur10/collision/wrist1.stl; visual mesh filename=../assets/ur10/official/meshes/ur10/visual/wrist1.dae
- link wrist_2_link: mass 1.96 -> 2.0; geometry collision mesh filename=../assets/ur10/official/meshes/ur10/collision/wrist2.stl; visual mesh filename=../assets/ur10/official/meshes/ur10/visual/wrist2.dae
- link wrist_3_link: mass 0.202 -> 0.365; geometry collision mesh filename=../assets/ur10/official/meshes/ur10/collision/wrist3.stl; visual mesh filename=../assets/ur10/official/meshes/ur10/visual/wrist3.dae
Joints:
- removed joint ee_fixed_joint
- removed joint world_joint
- removed joint wrist_3_link-tool0_fixed_joint
- added joint base_joint: type fixed, parent world, child base_link, origin xyz=0 0 0 rpy=0 0 0
- added joint base_link-base_link_inertia: type fixed, parent base_link, child base_link_inertia, origin xyz=0 0 0 rpy=0 0 3.141592653589793
- added joint flange-tool0: type fixed, parent flange, child tool0, origin xyz=0 0 0 rpy=1.5707963267948966 0 1.5707963267948966
- added joint wrist_3-flange: type fixed, parent wrist_3_link, child flange, origin xyz=0 0 0 rpy=0 -1.5707963267948966 -1.5707963267948966
- added joint wrist_3_link-ft_frame: type fixed, parent wrist_3_link, child ft_frame, origin xyz=0 0 0 rpy=3.141592653589793 0 0
- joint base_link-base_fixed_joint: origin xyz=0 0 0 rpy=0 0 -3.14159265359 -> xyz=0 0 0 rpy=0 0 3.141592653589793
- joint elbow_joint: axis 0 1 0 -> 0 0 1; limit lower=-3.14159265359 upper=3.14159265359 effort=150.0 velocity=3.15 -> lower=-3.141592653589793 upper=3.141592653589793 effort=150.0 velocity=3.141592653589793; origin xyz=0.0 -0.1719 0.612 rpy=0.0 0.0 0.0 -> xyz=-0.612 0 0 rpy=0 0 0
- joint shoulder_lift_joint: axis 0 1 0 -> 0 0 1; limit lower=-6.28318530718 upper=6.28318530718 effort=330.0 velocity=2.16 -> lower=-6.283185307179586 upper=6.283185307179586 effort=330.0 velocity=2.0943951023931953; origin xyz=0.0 0.220941 0.0 rpy=0.0 1.57079632679 0.0 -> xyz=0 0 0 rpy=1.570796327 0 0
- joint shoulder_pan_joint: limit lower=-6.28318530718 upper=6.28318530718 effort=330.0 velocity=2.16 -> lower=-6.283185307179586 upper=6.283185307179586 effort=330.0 velocity=2.0943951023931953; origin xyz=0.0 0.0 0.1273 rpy=0.0 0.0 0.0 -> xyz=0 0 0.1273 rpy=0 0 0; parent base_link -> base_link_inertia
- joint wrist_1_joint: axis 0 1 0 -> 0 0 1; limit lower=-6.28318530718 upper=6.28318530718 effort=54.0 velocity=3.2 -> lower=-6.283185307179586 upper=6.283185307179586 effort=56.0 velocity=3.141592653589793; origin xyz=0.0 0.0 0.5723 rpy=0.0 1.57079632679 0.0 -> xyz=-0.5723 0 0.163941 rpy=0 0 0
- joint wrist_2_joint: limit lower=-6.28318530718 upper=6.28318530718 effort=54.0 velocity=3.2 -> lower=-6.283185307179586 upper=6.283185307179586 effort=56.0 velocity=3.141592653589793; origin xyz=0.0 0.1149 0.0 rpy=0.0 0.0 0.0 -> xyz=0 -0.1157 -2.373046667922381e-11 rpy=1.570796327 0 0
- joint wrist_3_joint: axis 0 1 0 -> 0 0 1; limit lower=-6.28318530718 upper=6.28318530718 effort=54.0 velocity=3.2 -> lower=-6.283185307179586 upper=6.283185307179586 effort=56.0 velocity=3.141592653589793; origin xyz=0.0 0.0 0.1157 rpy=0.0 0.0 0.0 -> xyz=0 0.0922 -1.891053610911353e-11 rpy=1.570796326589793 3.141592653589793 3.141592653589793

File: script/ikea_table_prototype/generated/ur10_robotiq.urdf (robot description, URDF)
Before this commit: robot ur10_robotiq, 24 links, 23 joints
Links:
- removed link ee_link
- added link base_link_inertia, mass 4.0; collision mesh filename=../assets/ur10/official/meshes/ur10/collision/base.stl; visual mesh filename=../assets/ur10/official/meshes/ur10/visual/base.dae
- added link flange
- added link ft_frame
- link base: mass 0.0 -> None
- link base_link: mass 4.0 -> None; geometry 
- link forearm_link: mass 3.87 -> 4.27; geometry collision mesh filename=../assets/ur10/official/meshes/ur10/collision/forearm.stl; visual mesh filename=../assets/ur10/official/meshes/ur10/visual/forearm.dae
- link shoulder_link: mass 7.778 -> 7.1; geometry collision mesh filename=../assets/ur10/official/meshes/ur10/collision/shoulder.stl; visual mesh filename=../assets/ur10/official/meshes/ur10/visual/shoulder.dae
- link tool0: mass 0.0 -> None
- link upper_arm_link: mass 12.93 -> 12.7; geometry collision mesh filename=../assets/ur10/official/meshes/ur10/collision/upperarm.stl; visual mesh filename=../assets/ur10/official/meshes/ur10/visual/upperarm.dae
- link wrist_1_link: mass 1.96 -> 2.0; geometry collision mesh filename=../assets/ur10/official/meshes/ur10/collision/wrist1.stl; visual mesh filename=../assets/ur10/official/meshes/ur10/visual/wrist1.dae
- link wrist_2_link: mass 1.96 -> 2.0; geometry collision mesh filename=../assets/ur10/official/meshes/ur10/collision/wrist2.stl; visual mesh filename=../assets/ur10/official/meshes/ur10/visual/wrist2.dae
- link wrist_3_link: mass 0.202 -> 0.365; geometry collision mesh filename=../assets/ur10/official/meshes/ur10/collision/wrist3.stl; visual mesh filename=../assets/ur10/official/meshes/ur10/visual/wrist3.dae
Joints:
- removed joint ee_fixed_joint
- removed joint world_joint
- removed joint wrist_3_link-tool0_fixed_joint
- added joint base_joint: type fixed, parent world, child base_link, origin xyz=0 0 0 rpy=0 0 0
- added joint base_link-base_link_inertia: type fixed, parent base_link, child base_link_inertia, origin xyz=0 0 0 rpy=0 0 3.141592653589793
- added joint flange-tool0: type fixed, parent flange, child tool0, origin xyz=0 0 0 rpy=1.5707963267948966 0 1.5707963267948966
- added joint wrist_3-flange: type fixed, parent wrist_3_link, child flange, origin xyz=0 0 0 rpy=0 -1.5707963267948966 -1.5707963267948966
- added joint wrist_3_link-ft_frame: type fixed, parent wrist_3_link, child ft_frame, origin xyz=0 0 0 rpy=3.141592653589793 0 0
- joint base_link-base_fixed_joint: origin xyz=0 0 0 rpy=0 0 -3.14159265359 -> xyz=0 0 0 rpy=0 0 3.141592653589793
- joint elbow_joint: axis 0 1 0 -> 0 0 1; limit lower=-3.14159265359 upper=3.14159265359 effort=150.0 velocity=3.15 -> lower=-3.141592653589793 upper=3.141592653589793 effort=150.0 velocity=3.141592653589793; origin xyz=0.0 -0.1719 0.612 rpy=0.0 0.0 0.0 -> xyz=-0.612 0 0 rpy=0 0 0
- joint shoulder_lift_joint: axis 0 1 0 -> 0 0 1; limit lower=-6.28318530718 upper=6.28318530718 effort=330.0 velocity=2.16 -> lower=-6.283185307179586 upper=6.283185307179586 effort=330.0 velocity=2.0943951023931953; origin xyz=0.0 0.220941 0.0 rpy=0.0 1.57079632679 0.0 -> xyz=0 0 0 rpy=1.570796327 0 0
- joint shoulder_pan_joint: limit lower=-6.28318530718 upper=6.28318530718 effort=330.0 velocity=2.16 -> lower=-6.283185307179586 upper=6.283185307179586 effort=330.0 velocity=2.0943951023931953; origin xyz=0.0 0.0 0.1273 rpy=0.0 0.0 0.0 -> xyz=0 0 0.1273 rpy=0 0 0; parent base_link -> base_link_inertia
- joint wrist_1_joint: axis 0 1 0 -> 0 0 1; limit lower=-6.28318530718 upper=6.28318530718 effort=54.0 velocity=3.2 -> lower=-6.283185307179586 upper=6.283185307179586 effort=56.0 velocity=3.141592653589793; origin xyz=0.0 0.0 0.5723 rpy=0.0 1.57079632679 0.0 -> xyz=-0.5723 0 0.163941 rpy=0 0 0
- joint wrist_2_joint: limit lower=-6.28318530718 upper=6.28318530718 effort=54.0 velocity=3.2 -> lower=-6.283185307179586 upper=6.283185307179586 effort=56.0 velocity=3.141592653589793; origin xyz=0.0 0.1149 0.0 rpy=0.0 0.0 0.0 -> xyz=0 -0.1157 -2.373046667922381e-11 rpy=1.570796327 0 0
- joint wrist_3_joint: axis 0 1 0 -> 0 0 1; limit lower=-6.28318530718 upper=6.28318530718 effort=54.0 velocity=3.2 -> lower=-6.283185307179586 upper=6.283185307179586 effort=56.0 velocity=3.141592653589793; origin xyz=0.0 0.0 0.1157 rpy=0.0 0.0 0.0 -> xyz=0 0.0922 -1.891053610911353e-11 rpy=1.570796326589793 3.141592653589793 3.141592653589793

File: script/ikea_table_prototype/generated/ur10_robotiq_right.container.urdf (robot description, URDF)
Before this commit: robot ur10_robotiq, 25 links, 24 joints
Links:
- removed link ee_link
- added link base_link_inertia, mass 4.0; collision mesh filename=../assets/ur10/official/meshes/ur10/collision/base.stl; visual mesh filename=../assets/ur10/official/meshes/ur10/visual/base.dae
- added link flange
- added link ft_frame
- link base: mass 0.0 -> None
- link base_link: mass 4.0 -> None; geometry 
- link forearm_link: mass 3.87 -> 4.27; geometry collision mesh filename=../assets/ur10/official/meshes/ur10/collision/forearm.stl; visual mesh filename=../assets/ur10/official/meshes/ur10/visual/forearm.dae
- link shoulder_link: mass 7.778 -> 7.1; geometry collision mesh filename=../assets/ur10/official/meshes/ur10/collision/shoulder.stl; visual mesh filename=../assets/ur10/official/meshes/ur10/visual/shoulder.dae
- link tool0: mass 0.0 -> None
- link upper_arm_link: mass 12.93 -> 12.7; geometry collision mesh filename=../assets/ur10/official/meshes/ur10/collision/upperarm.stl; visual mesh filename=../assets/ur10/official/meshes/ur10/visual/upperarm.dae
- link wrist_1_link: mass 1.96 -> 2.0; geometry collision mesh filename=../assets/ur10/official/meshes/ur10/collision/wrist1.stl; visual mesh filename=../assets/ur10/official/meshes/ur10/visual/wrist1.dae
- link wrist_2_link: mass 1.96 -> 2.0; geometry collision mesh filename=../assets/ur10/official/meshes/ur10/collision/wrist2.stl; visual mesh filename=../assets/ur10/official/meshes/ur10/visual/wrist2.dae
- link wrist_3_link: mass 0.202 -> 0.365; geometry collision mesh filename=../assets/ur10/official/meshes/ur10/collision/wrist3.stl; visual mesh filename=../assets/ur10/official/meshes/ur10/visual/wrist3.dae
Joints:
- removed joint ee_fixed_joint
- removed joint world_joint
- removed joint wrist_3_link-tool0_fixed_joint
- added joint base_joint: type fixed, parent world, child base_link, origin xyz=0 0 0 rpy=0 0 0
- added joint base_link-base_link_inertia: type fixed, parent base_link, child base_link_inertia, origin xyz=0 0 0 rpy=0 0 3.141592653589793
- added joint flange-tool0: type fixed, parent flange, child tool0, origin xyz=0 0 0 rpy=1.5707963267948966 0 1.5707963267948966
- added joint wrist_3-flange: type fixed, parent wrist_3_link, child flange, origin xyz=0 0 0 rpy=0 -1.5707963267948966 -1.5707963267948966
- added joint wrist_3_link-ft_frame: type fixed, parent wrist_3_link, child ft_frame, origin xyz=0 0 0 rpy=3.141592653589793 0 0
- joint base_link-base_fixed_joint: origin xyz=0 0 0 rpy=0 0 -3.14159265359 -> xyz=0 0 0 rpy=0 0 3.141592653589793
- joint elbow_joint: axis 0 1 0 -> 0 0 1; limit lower=-3.14159265359 upper=3.14159265359 effort=150.0 velocity=3.15 -> lower=-3.141592653589793 upper=3.141592653589793 effort=150.0 velocity=3.141592653589793; origin xyz=0.0 -0.1719 0.612 rpy=0.0 0.0 0.0 -> xyz=-0.612 0 0 rpy=0 0 0
- joint shoulder_lift_joint: axis 0 1 0 -> 0 0 1; limit lower=-6.28318530718 upper=6.28318530718 effort=330.0 velocity=2.16 -> lower=-6.283185307179586 upper=6.283185307179586 effort=330.0 velocity=2.0943951023931953; origin xyz=0.0 0.220941 0.0 rpy=0.0 1.57079632679 0.0 -> xyz=0 0 0 rpy=1.570796327 0 0
- joint shoulder_pan_joint: limit lower=-6.28318530718 upper=6.28318530718 effort=330.0 velocity=2.16 -> lower=-6.283185307179586 upper=6.283185307179586 effort=330.0 velocity=2.0943951023931953; origin xyz=0.0 0.0 0.1273 rpy=0.0 0.0 0.0 -> xyz=0 0 0.1273 rpy=0 0 0; parent base_link -> base_link_inertia
- joint wrist_1_joint: axis 0 1 0 -> 0 0 1; limit lower=-6.28318530718 upper=6.28318530718 effort=54.0 velocity=3.2 -> lower=-6.283185307179586 upper=6.283185307179586 effort=56.0 velocity=3.141592653589793; origin xyz=0.0 0.0 0.5723 rpy=0.0 1.57079632679 0.0 -> xyz=-0.5723 0 0.163941 rpy=0 0 0
- joint wrist_2_joint: limit lower=-6.28318530718 upper=6.28318530718 effort=54.0 velocity=3.2 -> lower=-6.283185307179586 upper=6.283185307179586 effort=56.0 velocity=3.141592653589793; origin xyz=0.0 0.1149 0.0 rpy=0.0 0.0 0.0 -> xyz=0 -0.1157 -2.373046667922381e-11 rpy=1.570796327 0 0
- joint wrist_3_joint: axis 0 1 0 -> 0 0 1; limit lower=-6.28318530718 upper=6.28318530718 effort=54.0 velocity=3.2 -> lower=-6.283185307179586 upper=6.283185307179586 effort=56.0 velocity=3.141592653589793; origin xyz=0.0 0.0 0.1157 rpy=0.0 0.0 0.0 -> xyz=0 0.0922 -1.891053610911353e-11 rpy=1.570796326589793 3.141592653589793 3.141592653589793

File: script/ikea_table_prototype/generated/ur10_robotiq_right.urdf (robot description, URDF)
Before this commit: robot ur10_robotiq, 25 links, 24 joints
Links:
- removed link ee_link
- added link base_link_inertia, mass 4.0; collision mesh filename=../assets/ur10/official/meshes/ur10/collision/base.stl; visual mesh filename=../assets/ur10/official/meshes/ur10/visual/base.dae
- added link flange
- added link ft_frame
- link base: mass 0.0 -> None
- link base_link: mass 4.0 -> None; geometry 
- link forearm_link: mass 3.87 -> 4.27; geometry collision mesh filename=../assets/ur10/official/meshes/ur10/collision/forearm.stl; visual mesh filename=../assets/ur10/official/meshes/ur10/visual/forearm.dae
- link shoulder_link: mass 7.778 -> 7.1; geometry collision mesh filename=../assets/ur10/official/meshes/ur10/collision/shoulder.stl; visual mesh filename=../assets/ur10/official/meshes/ur10/visual/shoulder.dae
- link tool0: mass 0.0 -> None
- link upper_arm_link: mass 12.93 -> 12.7; geometry collision mesh filename=../assets/ur10/official/meshes/ur10/collision/upperarm.stl; visual mesh filename=../assets/ur10/official/meshes/ur10/visual/upperarm.dae
- link wrist_1_link: mass 1.96 -> 2.0; geometry collision mesh filename=../assets/ur10/official/meshes/ur10/collision/wrist1.stl; visual mesh filename=../assets/ur10/official/meshes/ur10/visual/wrist1.dae
- link wrist_2_link: mass 1.96 -> 2.0; geometry collision mesh filename=../assets/ur10/official/meshes/ur10/collision/wrist2.stl; visual mesh filename=../assets/ur10/official/meshes/ur10/visual/wrist2.dae
- link wrist_3_link: mass 0.202 -> 0.365; geometry collision mesh filename=../assets/ur10/official/meshes/ur10/collision/wrist3.stl; visual mesh filename=../assets/ur10/official/meshes/ur10/visual/wrist3.dae
Joints:
- removed joint ee_fixed_joint
- removed joint world_joint
- removed joint wrist_3_link-tool0_fixed_joint
- added joint base_joint: type fixed, parent world, child base_link, origin xyz=0 0 0 rpy=0 0 0
- added joint base_link-base_link_inertia: type fixed, parent base_link, child base_link_inertia, origin xyz=0 0 0 rpy=0 0 3.141592653589793
- added joint flange-tool0: type fixed, parent flange, child tool0, origin xyz=0 0 0 rpy=1.5707963267948966 0 1.5707963267948966
- added joint wrist_3-flange: type fixed, parent wrist_3_link, child flange, origin xyz=0 0 0 rpy=0 -1.5707963267948966 -1.5707963267948966
- added joint wrist_3_link-ft_frame: type fixed, parent wrist_3_link, child ft_frame, origin xyz=0 0 0 rpy=3.141592653589793 0 0
- joint base_link-base_fixed_joint: origin xyz=0 0 0 rpy=0 0 -3.14159265359 -> xyz=0 0 0 rpy=0 0 3.141592653589793
- joint elbow_joint: axis 0 1 0 -> 0 0 1; limit lower=-3.14159265359 upper=3.14159265359 effort=150.0 velocity=3.15 -> lower=-3.141592653589793 upper=3.141592653589793 effort=150.0 velocity=3.141592653589793; origin xyz=0.0 -0.1719 0.612 rpy=0.0 0.0 0.0 -> xyz=-0.612 0 0 rpy=0 0 0
- joint shoulder_lift_joint: axis 0 1 0 -> 0 0 1; limit lower=-6.28318530718 upper=6.28318530718 effort=330.0 velocity=2.16 -> lower=-6.283185307179586 upper=6.283185307179586 effort=330.0 velocity=2.0943951023931953; origin xyz=0.0 0.220941 0.0 rpy=0.0 1.57079632679 0.0 -> xyz=0 0 0 rpy=1.570796327 0 0
- joint shoulder_pan_joint: limit lower=-6.28318530718 upper=6.28318530718 effort=330.0 velocity=2.16 -> lower=-6.283185307179586 upper=6.283185307179586 effort=330.0 velocity=2.0943951023931953; origin xyz=0.0 0.0 0.1273 rpy=0.0 0.0 0.0 -> xyz=0 0 0.1273 rpy=0 0 0; parent base_link -> base_link_inertia
- joint wrist_1_joint: axis 0 1 0 -> 0 0 1; limit lower=-6.28318530718 upper=6.28318530718 effort=54.0 velocity=3.2 -> lower=-6.283185307179586 upper=6.283185307179586 effort=56.0 velocity=3.141592653589793; origin xyz=0.0 0.0 0.5723 rpy=0.0 1.57079632679 0.0 -> xyz=-0.5723 0 0.163941 rpy=0 0 0
- joint wrist_2_joint: limit lower=-6.28318530718 upper=6.28318530718 effort=54.0 velocity=3.2 -> lower=-6.283185307179586 upper=6.283185307179586 effort=56.0 velocity=3.141592653589793; origin xyz=0.0 0.1149 0.0 rpy=0.0 0.0 0.0 -> xyz=0 -0.1157 -2.373046667922381e-11 rpy=1.570796327 0 0
- joint wrist_3_joint: axis 0 1 0 -> 0 0 1; limit lower=-6.28318530718 upper=6.28318530718 effort=54.0 velocity=3.2 -> lower=-6.283185307179586 upper=6.283185307179586 effort=56.0 velocity=3.141592653589793; origin xyz=0.0 0.0 0.1157 rpy=0.0 0.0 0.0 -> xyz=0 0.0922 -1.891053610911353e-11 rpy=1.570796326589793 3.141592653589793 3.141592653589793
