Commit message: feat(examples): the Robotiq 2F-85 from PickNik's ros2_robotiq_gripper (#71)

File: script/ikea_table_prototype/generated/ur10_robotiq.container.urdf (robot description, URDF)
Before this commit: robot ur10_robotiq, 26 links, 25 joints
Links:
- removed link left_inner_finger
- removed link left_inner_finger_pad
- removed link left_inner_knuckle
- removed link left_outer_finger
- removed link left_outer_knuckle
- removed link right_inner_finger
- removed link right_inner_finger_pad
- removed link right_inner_knuckle
- removed link right_outer_finger
- removed link right_outer_knuckle
- removed link robotiq_arg2f_base_link
- added link robotiq_85_base_link, mass 6.6320197e-01; collision mesh filename=../assets/robotiq_2f85/picknik/meshes/collision/2f_85/robot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; visual mesh filename=../assets/robotiq_2f85/picknik/meshes/visual/2f_85/robotiq_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
- added link robotiq_85_left_finger_link, mass 4.260376752e-02; collision mesh filename=../assets/robotiq_2f85/picknik/meshes/collision/2f_85/left_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; visual mesh filename=../assets/robotiq_2f85/picknik/meshes/visual/2f_85/left_fin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
- added link robotiq_85_left_finger_pad
- added link robotiq_85_left_finger_tip_link, mass 4.268588744e-02; collision mesh filename=../assets/robotiq_2f85/picknik/meshes/collision/2f_85/left_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; visual mesh filename=../assets/robotiq_2f85/picknik/meshes/visual/2f_85/left_fin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
- added link robotiq_85_left_inner_knuckle_link, mass 2.969376448e-02; collision mesh filename=../assets/robotiq_2f85/picknik/meshes/collision/2f_85/left_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; visual mesh filename=../assets/robotiq_2f85/picknik/meshes/visual/2f_85/left_inn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
- added link robotiq_85_left_knuckle_link, mass 1.384773208e-02; collision mesh filename=../assets/robotiq_2f85/picknik/meshes/collision/2f_85/left_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; visual mesh filename=../assets/robotiq_2f85/picknik/meshes/visual/2f_85/left_knu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
- added link robotiq_85_right_finger_link, mass 4.260376752000000e-02; collision mesh filename=../assets/robotiq_2f85/picknik/meshes/collision/2f_85/right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; visual mesh filename=../assets/robotiq_2f85/picknik/meshes/visual/2f_85/right_fi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
- added link robotiq_85_right_finger_pad
- added link robotiq_85_right_finger_tip_link, mass 4.268588744e-02; collision mesh filename=../assets/robotiq_2f85/picknik/meshes/collision/2f_85/right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; visual mesh filename=../assets/robotiq_2f85/picknik/meshes/visual/2f_85/right_fi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
- added link robotiq_85_right_inner_knuckle_link, mass 2.969376448e-02; collision mesh filename=../assets/robotiq_2f85/picknik/meshes/collision/2f_85/right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; visual mesh filename=../assets/robotiq_2f85/picknik/meshes/visual/2f_85/right_in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
- added link robotiq_85_right_knuckle_link, mass 1.384773208e-02; collision mesh filename=../assets/robotiq_2f85/picknik/meshes/collision/2f_85/right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; visual mesh filename=../assets/robotiq_2f85/picknik/meshes/visual/2f_85/right_kn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
Joints:
- removed joint finger_joint
- removed joint left_inner_finger_joint
- removed joint left_inner_finger_pad_joint
- removed joint left_inner_knuckle_joint
- removed joint left_outer_finger_joint
- removed joint right_inner_finger_joint
- removed joint right_inner_finger_pad_joint
- removed joint right_inner_knuckle_joint
- removed joint right_outer_finger_joint
- removed joint right_outer_knuckle_joint
- added joint robotiq_85_left_finger_joint: type fixed, parent robotiq_85_left_knuckle_link, child robotiq_85_left_finger_link, origin xyz=0.03152616 0.0 -0.00376347 rpy=0 0 0
- added joint robotiq_85_left_finger_pad_joint: type fixed, parent robotiq_85_left_finger_tip_link, child robotiq_85_left_finger_pad, origin xyz=-0.0253 0 0.032 rpy=0 0 0
- added joint robotiq_85_left_finger_tip_joint: type revolute, parent robotiq_85_left_finger_link, child robotiq_85_left_finger_tip_link, origin xyz=0.00563134 0.0 0.04718515 rpy=0 0 0, axis 0 -1 0, limit lower=-0.8 upper=0.0 effort=50 velocity=0.5, mimic joint=robotiq_85_left_knuckle_joint multiplier=-1
- added joint robotiq_85_left_inner_knuckle_joint: type revolute, parent robotiq_85_base_link, child robotiq_85_left_inner_knuckle_link, origin xyz=0.0127 0.0 0.06142 rpy=0 0 0, axis 0 -1 0, limit lower=0.0 upper=0.8 effort=50 velocity=0.5, mimic joint=robotiq_85_left_knuckle_joint
- added joint robotiq_85_left_knuckle_joint: type revolute, parent robotiq_85_base_link, child robotiq_85_left_knuckle_link, origin xyz=0.03060114 0.0 0.05490452 rpy=0 0 0, axis 0 -1 0, limit lower=0.0 upper=0.8 effort=50 velocity=0.5
- added joint robotiq_85_right_finger_joint: type fixed, parent robotiq_85_right_knuckle_link, child robotiq_85_right_finger_link, origin xyz=-0.03152616 0.0 -0.00376347 rpy=0 0 0
- added joint robotiq_85_right_finger_pad_joint: type fixed, parent robotiq_85_right_finger_tip_link, child robotiq_85_right_finger_pad, origin xyz=0.0253 0 0.032 rpy=0 0 0
- added joint robotiq_85_right_finger_tip_joint: type revolute, parent robotiq_85_right_finger_link, child robotiq_85_right_finger_tip_link, origin xyz=-0.00563134 0.0 0.04718515 rpy=0 0 0, axis 0 -1 0, limit lower=0.0 upper=0.8 effort=50 velocity=0.5, mimic joint=robotiq_85_left_knuckle_joint
- added joint robotiq_85_right_inner_knuckle_joint: type revolute, parent robotiq_85_base_link, child robotiq_85_right_inner_knuckle_link, origin xyz=-0.0127 0.0 0.06142 rpy=0 0 0, axis 0 -1 0, limit lower=-0.8 upper=0.0 effort=50 velocity=0.5, mimic joint=robotiq_85_left_knuckle_joint multiplier=-1
- added joint robotiq_85_right_knuckle_joint: type revolute, parent robotiq_85_base_link, child robotiq_85_right_knuckle_link, origin xyz=-0.03060114 0.0 0.05490452 rpy=0 0 0, axis 0 -1 0, limit lower=-0.8 upper=0.0 effort=50 velocity=0.5, mimic joint=robotiq_85_left_knuckle_joint multiplier=-1
- joint gripper_to_tcp: origin xyz=0 0 0.15 rpy=0 0 0 -> xyz=0 0 0.15 rpy=0 0 1.5707963267948966; parent robotiq_arg2f_base_link -> robotiq_85_base_link
- joint tool0_to_gripper: child robotiq_arg2f_base_link -> robotiq_85_base_link; origin xyz=0 0 0 rpy=0 0 0 -> xyz=0 0 0 rpy=0 0 -1.5707963267948966

File: script/ikea_table_prototype/generated/ur10_robotiq.urdf (robot description, URDF)
Before this commit: robot ur10_robotiq, 26 links, 25 joints
Links:
- removed link left_inner_finger
- removed link left_inner_finger_pad
- removed link left_inner_knuckle
- removed link left_outer_finger
- removed link left_outer_knuckle
- removed link right_inner_finger
- removed link right_inner_finger_pad
- removed link right_inner_knuckle
- removed link right_outer_finger
- removed link right_outer_knuckle
- removed link robotiq_arg2f_base_link
- added link robotiq_85_base_link, mass 6.6320197e-01; collision mesh filename=../assets/robotiq_2f85/picknik/meshes/collision/2f_85/robot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; visual mesh filename=../assets/robotiq_2f85/picknik/meshes/visual/2f_85/robotiq_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
- added link robotiq_85_left_finger_link, mass 4.260376752e-02; collision mesh filename=../assets/robotiq_2f85/picknik/meshes/collision/2f_85/left_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; visual mesh filename=../assets/robotiq_2f85/picknik/meshes/visual/2f_85/left_fin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
- added link robotiq_85_left_finger_pad
- added link robotiq_85_left_finger_tip_link, mass 4.268588744e-02; collision mesh filename=../assets/robotiq_2f85/picknik/meshes/collision/2f_85/left_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; visual mesh filename=../assets/robotiq_2f85/picknik/meshes/visual/2f_85/left_fin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
- added link robotiq_85_left_inner_knuckle_link, mass 2.969376448e-02; collision mesh filename=../assets/robotiq_2f85/picknik/meshes/collision/2f_85/left_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; visual mesh filename=../assets/robotiq_2f85/picknik/meshes/visual/2f_85/left_inn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
- added link robotiq_85_left_knuckle_link, mass 1.384773208e-02; collision mesh filename=../assets/robotiq_2f85/picknik/meshes/collision/2f_85/left_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; visual mesh filename=../assets/robotiq_2f85/picknik/meshes/visual/2f_85/left_knu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
- added link robotiq_85_right_finger_link, mass 4.260376752000000e-02; collision mesh filename=../assets/robotiq_2f85/picknik/meshes/collision/2f_85/right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; visual mesh filename=../assets/robotiq_2f85/picknik/meshes/visual/2f_85/right_fi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
- added link robotiq_85_right_finger_pad
- added link robotiq_85_right_finger_tip_link, mass 4.268588744e-02; collision mesh filename=../assets/robotiq_2f85/picknik/meshes/collision/2f_85/right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; visual mesh filename=../assets/robotiq_2f85/picknik/meshes/visual/2f_85/right_fi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
- added link robotiq_85_right_inner_knuckle_link, mass 2.969376448e-02; collision mesh filename=../assets/robotiq_2f85/picknik/meshes/collision/2f_85/right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; visual mesh filename=../assets/robotiq_2f85/picknik/meshes/visual/2f_85/right_in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
- added link robotiq_85_right_knuckle_link, mass 1.384773208e-02; collision mesh filename=../assets/robotiq_2f85/picknik/meshes/collision/2f_85/right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; visual mesh filename=../assets/robotiq_2f85/picknik/meshes/visual/2f_85/right_kn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
Joints:
- removed joint finger_joint
- removed joint left_inner_finger_joint
- removed joint left_inner_finger_pad_joint
- removed joint left_inner_knuckle_joint
- removed joint left_outer_finger_joint
- removed joint right_inner_finger_joint
- removed joint right_inner_finger_pad_joint
- removed joint right_inner_knuckle_joint
- removed joint right_outer_finger_joint
- removed joint right_outer_knuckle_joint
- added joint robotiq_85_left_finger_joint: type fixed, parent robotiq_85_left_knuckle_link, child robotiq_85_left_finger_link, origin xyz=0.03152616 0.0 -0.00376347 rpy=0 0 0
- added joint robotiq_85_left_finger_pad_joint: type fixed, parent robotiq_85_left_finger_tip_link, child robotiq_85_left_finger_pad, origin xyz=-0.0253 0 0.032 rpy=0 0 0
- added joint robotiq_85_left_finger_tip_joint: type revolute, parent robotiq_85_left_finger_link, child robotiq_85_left_finger_tip_link, origin xyz=0.00563134 0.0 0.04718515 rpy=0 0 0, axis 0 -1 0, limit lower=-0.8 upper=0.0 effort=50 velocity=0.5, mimic joint=robotiq_85_left_knuckle_joint multiplier=-1
- added joint robotiq_85_left_inner_knuckle_joint: type revolute, parent robotiq_85_base_link, child robotiq_85_left_inner_knuckle_link, origin xyz=0.0127 0.0 0.06142 rpy=0 0 0, axis 0 -1 0, limit lower=0.0 upper=0.8 effort=50 velocity=0.5, mimic joint=robotiq_85_left_knuckle_joint
- added joint robotiq_85_left_knuckle_joint: type revolute, parent robotiq_85_base_link, child robotiq_85_left_knuckle_link, origin xyz=0.03060114 0.0 0.05490452 rpy=0 0 0, axis 0 -1 0, limit lower=0.0 upper=0.8 effort=50 velocity=0.5
- added joint robotiq_85_right_finger_joint: type fixed, parent robotiq_85_right_knuckle_link, child robotiq_85_right_finger_link, origin xyz=-0.03152616 0.0 -0.00376347 rpy=0 0 0
- added joint robotiq_85_right_finger_pad_joint: type fixed, parent robotiq_85_right_finger_tip_link, child robotiq_85_right_finger_pad, origin xyz=0.0253 0 0.032 rpy=0 0 0
- added joint robotiq_85_right_finger_tip_joint: type revolute, parent robotiq_85_right_finger_link, child robotiq_85_right_finger_tip_link, origin xyz=-0.00563134 0.0 0.04718515 rpy=0 0 0, axis 0 -1 0, limit lower=0.0 upper=0.8 effort=50 velocity=0.5, mimic joint=robotiq_85_left_knuckle_joint
- added joint robotiq_85_right_inner_knuckle_joint: type revolute, parent robotiq_85_base_link, child robotiq_85_right_inner_knuckle_link, origin xyz=-0.0127 0.0 0.06142 rpy=0 0 0, axis 0 -1 0, limit lower=-0.8 upper=0.0 effort=50 velocity=0.5, mimic joint=robotiq_85_left_knuckle_joint multiplier=-1
- added joint robotiq_85_right_knuckle_joint: type revolute, parent robotiq_85_base_link, child robotiq_85_right_knuckle_link, origin xyz=-0.03060114 0.0 0.05490452 rpy=0 0 0, axis 0 -1 0, limit lower=-0.8 upper=0.0 effort=50 velocity=0.5, mimic joint=robotiq_85_left_knuckle_joint multiplier=-1
- joint gripper_to_tcp: origin xyz=0 0 0.15 rpy=0 0 0 -> xyz=0 0 0.15 rpy=0 0 1.5707963267948966; parent robotiq_arg2f_base_link -> robotiq_85_base_link
- joint tool0_to_gripper: child robotiq_arg2f_base_link -> robotiq_85_base_link; origin xyz=0 0 0 rpy=0 0 0 -> xyz=0 0 0 rpy=0 0 -1.5707963267948966

File: script/ikea_table_prototype/generated/ur10_robotiq_right.container.urdf (robot description, URDF)
Before this commit: robot ur10_robotiq, 27 links, 26 joints
Links:
- removed link left_inner_finger
- removed link left_inner_finger_pad
- removed link left_inner_knuckle
- removed link left_outer_finger
- removed link left_outer_knuckle
- removed link right_inner_finger
- removed link right_inner_finger_pad
- removed link right_inner_knuckle
- removed link right_outer_finger
- removed link right_outer_knuckle
- removed link robotiq_arg2f_base_link
- added link robotiq_85_base_link, mass 6.6320197e-01; collision mesh filename=../assets/robotiq_2f85/picknik/meshes/collision/2f_85/robot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; visual mesh filename=../assets/robotiq_2f85/picknik/meshes/visual/2f_85/robotiq_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
- added link robotiq_85_left_finger_link, mass 4.260376752e-02; collision mesh filename=../assets/robotiq_2f85/picknik/meshes/collision/2f_85/left_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; visual mesh filename=../assets/robotiq_2f85/picknik/meshes/visual/2f_85/left_fin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
- added link robotiq_85_left_finger_pad
- added link robotiq_85_left_finger_tip_link, mass 4.268588744e-02; collision mesh filename=../assets/robotiq_2f85/picknik/meshes/collision/2f_85/left_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; visual mesh filename=../assets/robotiq_2f85/picknik/meshes/visual/2f_85/left_fin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
- added link robotiq_85_left_inner_knuckle_link, mass 2.969376448e-02; collision mesh filename=../assets/robotiq_2f85/picknik/meshes/collision/2f_85/left_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; visual mesh filename=../assets/robotiq_2f85/picknik/meshes/visual/2f_85/left_inn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
- added link robotiq_85_left_knuckle_link, mass 1.384773208e-02; collision mesh filename=../assets/robotiq_2f85/picknik/meshes/collision/2f_85/left_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; visual mesh filename=../assets/robotiq_2f85/picknik/meshes/visual/2f_85/left_knu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
- added link robotiq_85_right_finger_link, mass 4.260376752000000e-02; collision mesh filename=../assets/robotiq_2f85/picknik/meshes/collision/2f_85/right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; visual mesh filename=../assets/robotiq_2f85/picknik/meshes/visual/2f_85/right_fi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
- added link robotiq_85_right_finger_pad
- added link robotiq_85_right_finger_tip_link, mass 4.268588744e-02; collision mesh filename=../assets/robotiq_2f85/picknik/meshes/collision/2f_85/right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; visual mesh filename=../assets/robotiq_2f85/picknik/meshes/visual/2f_85/right_fi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
- added link robotiq_85_right_inner_knuckle_link, mass 2.969376448e-02; collision mesh filename=../assets/robotiq_2f85/picknik/meshes/collision/2f_85/right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; visual mesh filename=../assets/robotiq_2f85/picknik/meshes/visual/2f_85/right_in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
- added link robotiq_85_right_knuckle_link, mass 1.384773208e-02; collision mesh filename=../assets/robotiq_2f85/picknik/meshes/collision/2f_85/right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; visual mesh filename=../assets/robotiq_2f85/picknik/meshes/visual/2f_85/right_kn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
Joints:
- removed joint finger_joint
- removed joint left_inner_finger_joint
- removed joint left_inner_finger_pad_joint
- removed joint left_inner_knuckle_joint
- removed joint left_outer_finger_joint
- removed joint right_inner_finger_joint
- removed joint right_inner_finger_pad_joint
- removed joint right_inner_knuckle_joint
- removed joint right_outer_finger_joint
- removed joint right_outer_knuckle_joint
- added joint robotiq_85_left_finger_joint: type fixed, parent robotiq_85_left_knuckle_link, child robotiq_85_left_finger_link, origin xyz=0.03152616 0.0 -0.00376347 rpy=0 0 0
- added joint robotiq_85_left_finger_pad_joint: type fixed, parent robotiq_85_left_finger_tip_link, child robotiq_85_left_finger_pad, origin xyz=-0.0253 0 0.032 rpy=0 0 0
- added joint robotiq_85_left_finger_tip_joint: type revolute, parent robotiq_85_left_finger_link, child robotiq_85_left_finger_tip_link, origin xyz=0.00563134 0.0 0.04718515 rpy=0 0 0, axis 0 -1 0, limit lower=-0.8 upper=0.0 effort=50 velocity=0.5, mimic joint=robotiq_85_left_knuckle_joint multiplier=-1
- added joint robotiq_85_left_inner_knuckle_joint: type revolute, parent robotiq_85_base_link, child robotiq_85_left_inner_knuckle_link, origin xyz=0.0127 0.0 0.06142 rpy=0 0 0, axis 0 -1 0, limit lower=0.0 upper=0.8 effort=50 velocity=0.5, mimic joint=robotiq_85_left_knuckle_joint
- added joint robotiq_85_left_knuckle_joint: type revolute, parent robotiq_85_base_link, child robotiq_85_left_knuckle_link, origin xyz=0.03060114 0.0 0.05490452 rpy=0 0 0, axis 0 -1 0, limit lower=0.0 upper=0.8 effort=50 velocity=0.5
- added joint robotiq_85_right_finger_joint: type fixed, parent robotiq_85_right_knuckle_link, child robotiq_85_right_finger_link, origin xyz=-0.03152616 0.0 -0.00376347 rpy=0 0 0
- added joint robotiq_85_right_finger_pad_joint: type fixed, parent robotiq_85_right_finger_tip_link, child robotiq_85_right_finger_pad, origin xyz=0.0253 0 0.032 rpy=0 0 0
- added joint robotiq_85_right_finger_tip_joint: type revolute, parent robotiq_85_right_finger_link, child robotiq_85_right_finger_tip_link, origin xyz=-0.00563134 0.0 0.04718515 rpy=0 0 0, axis 0 -1 0, limit lower=0.0 upper=0.8 effort=50 velocity=0.5, mimic joint=robotiq_85_left_knuckle_joint
- added joint robotiq_85_right_inner_knuckle_joint: type revolute, parent robotiq_85_base_link, child robotiq_85_right_inner_knuckle_link, origin xyz=-0.0127 0.0 0.06142 rpy=0 0 0, axis 0 -1 0, limit lower=-0.8 upper=0.0 effort=50 velocity=0.5, mimic joint=robotiq_85_left_knuckle_joint multiplier=-1
- added joint robotiq_85_right_knuckle_joint: type revolute, parent robotiq_85_base_link, child robotiq_85_right_knuckle_link, origin xyz=-0.03060114 0.0 0.05490452 rpy=0 0 0, axis 0 -1 0, limit lower=-0.8 upper=0.0 effort=50 velocity=0.5, mimic joint=robotiq_85_left_knuckle_joint multiplier=-1
- joint gripper_to_tcp: origin xyz=0 0 0.15 rpy=0 0 0 -> xyz=0 0 0.15 rpy=0 0 1.5707963267948966; parent robotiq_arg2f_base_link -> robotiq_85_base_link
- joint tool0_to_gripper: child robotiq_arg2f_base_link -> robotiq_85_base_link; origin xyz=0 0 0 rpy=0 0 0 -> xyz=0 0 0 rpy=0 0 -1.5707963267948966
