Commit message: docs(examples): ship the 4-part screw-assembly scene with its batch results
Regenerate the checked-in scene at the generator's default of 4 parts
and record the 10-seed batch it was validated on in the README:
10/10 missions completed, replanning trigger rate 0.0% (0/140 planning
blocks), recovery rate 100% (21/21, all by resuming), median mission
1223 s (579-2536 s), no native crashes. Also correct the block/phase
count formula (4N + 3 blocks; 7N + 3 grasp/release phases plus N + 1
home moves).

File: script/screw_assembly/generated/fixtures.urdf (robot description, URDF)
Before this commit: robot fixtures, 2 links, 1 joints
Links:
- link base_link: geometry collision box size=0.42 0.46 0.04; visual box size=0.42 0.46 0.04
