Commit message: feat(examples): make the screw-assembly driver a real cordless drill
Replace the 0.20 m cylinder screwdriver with the YCB 035_power_drill scan
(CC BY 4.0, vendored under assets/ycb_035_power_drill/ with attribution,
texture downscaled to 1024 px). The scan is the visual; collision is six
box/cylinder proxies fitted to it (battery, handle, trigger, body, chuck)
plus a 50 mm driver bit the scan lacks.

The Robotiq now grasps the handle the way a person holds a drill: it
approaches from behind along the bit and closes across the 38 mm handle.
The drill stands on its battery on a charging dock (the old tool rack,
now 0.14 x 0.09 x 0.03 m), bit pointing away from ur10_right. The tip
gripper is turned 180 deg about the bit so the handle points to +X world
while screwing, away from ur10_left's hand on the tab.

The mesh path follows the arms' convention (container-absolute);
build_scene.py --repo-root points it elsewhere. home_target() reads the
new DRIVER_GRIP_XYZQUAT.

Checked offline with pinocchio + coal only (no HPP): the open fingers
clear the handle by 24 mm at the grasp and 34 mm at the pregrasp, and
ur10_right has collision-free IK for the dock pick and all 8 holes.
The README's batch results predate this change and say so.

Co-Authored-By: Claude Opus 5.5 <noreply@anthropic.com>
Claude-Session: https://claude.ai/code/session_01JMeLhrREKP5sc7fCwNDVrr

File: script/screw_assembly/generated/driver.urdf (robot description, URDF)
Before this commit: robot driver, 1 links, 0 joints
Links:
- link base_link: mass 0.3 -> 0.895; geometry collision box size=0.04 0.038 0.04; collision box size=0.054 0.038 0.097

File: script/screw_assembly/generated/fixtures.urdf (robot description, URDF)
Before this commit: robot fixtures, 2 links, 1 joints
Links:
- link rack: geometry collision box size=0.14 0.09 0.03; visual box size=0.14 0.09 0.03

Commit message: feat(examples): load the IKEA and screw-assembly scenes from any checkout
The IKEA config names its URDFs relative to itself instead of by the
container path, and build_scene.py writes the drill mesh relative to
its URDF (--repo-root dropped). With the loader fixes, both scenes load
from a plain 'pip install -e .[hpp]' checkout: the screw-assembly
mission ran end to end (1 part, seed 2, 418 s) with no symlink and no
LD_LIBRARY_PATH. CHANGELOG and the screw-assembly README updated.

Co-Authored-By: Claude Opus 5.5 <noreply@anthropic.com>
Claude-Session: https://claude.ai/code/session_01JMeLhrREKP5sc7fCwNDVrr

File: script/screw_assembly/generated/driver.urdf (robot description, URDF)
Before this commit: robot driver, 1 links, 0 joints
Links:
- link base_link: geometry collision box size=0.04 0.038 0.04; collision box size=0.054 0.038 0.097
